File: Board/plantwatch.sch (KiCad schematic (older format))
At the start: 27 parts, among them J3 SWD Connector, J4 Jack-DC, SW1 SW_Push, SW2 SW_Push, U1 MKL25Z128VLK4, U4 NCP1117-3.3_SOT223, Y1 Crystal_GND24

Commit message: Make layout
Parts:
- C1, C7: value C_Small -> 0.2uF
Changed lines of the file:
@@
 P 8400 1550
 F 0 "C1" H 8492 1596 50  0000 L CNN
-F 1 "C_Small" H 8492 1505 50  0000 L CNN
+F 1 "0.2uF" H 8492 1505 50  0000 L CNN
 F 2 "Capacitor_THT:CP_Radial_Tantal_D4.5mm_P5.00mm" H 8400 1550 50  0001 C CNN
 F 3 "~" H 8400 1550 50  0001 C CNN
@@
 P 9600 1550
 F 0 "C7" H 9692 1596 50  0000 L CNN
-F 1 "C_Small" H 9692 1505 50  0000 L CNN
+F 1 "0.2uF" H 9692 1505 50  0000 L CNN
 F 2 "Capacitor_THT:CP_Radial_Tantal_D4.5mm_P5.00mm" H 9600 1550 50  0001 C CNN
 F 3 "~" H 9600 1550 50  0001 C CNN
@@
 	9800 1800 9600 1800
 Wire Wire Line
+	9800 1350 9800 1450
+Connection ~ 10000 1800
+Wire Wire Line
 	9600 1350 9800 1350
-Wire Wire Line
-	9800 1350 9800 1450
 Connection ~ 9800 1350
 Wire Wire Line
 	9800 1350 10000 1350
-Connection ~ 10000 1800
 $EndSCHEMATC

Commit message: PCB almost done
Parts:
- removed C14: 1uF, Capacitor_THT:CP_Radial_Tantal_D4.5mm_P5.00mm, symbol Device:C_Small
- removed C16: C_Small, Capacitor_THT:CP_Radial_Tantal_D4.5mm_P5.00mm, symbol Device:C_Small
- removed C7: 0.2uF, Capacitor_THT:CP_Radial_Tantal_D4.5mm_P5.00mm, symbol Device:C_Small
- removed J4: Jack-DC, symbol Connector:Jack-DC
- removed R9: 10K, Resistor_THT:R_Axial_DIN0411_L9.9mm_D3.6mm_P12.70mm_Horizontal, symbol Device:R_Small
- removed SW2: SW_Push, Button_Switch_THT:SW_PUSH_6mm, symbol Switch:SW_Push
- added J6: Power Input, Connector_BarrelJack:BarrelJack_Horizontal, symbol Connector:Barrel_Jack_Switch
- C1: value 0.2uF -> 0.1uF; footprint Capacitor_THT:CP_Radial_Tantal_D4.5mm_P5.00mm -> Capacitor_Tantalum_SMD:CP_EIA-3528-15_AVX-H_Pad1.50x2.35mm_HandSolder
- C12, C13, C8: footprint Capacitor_THT:CP_Radial_Tantal_D4.5mm_P5.00mm -> Capacitor_Tantalum_SMD:CP_EIA-3528-15_AVX-H_Pad1.50x2.35mm_HandSolder
- C15, C2, C3, C4, C5, C6: value C_Small -> 0.1uF; footprint Capacitor_THT:CP_Radial_Tantal_D4.5mm_P5.00mm -> Capacitor_Tantalum_SMD:CP_EIA-3528-15_AVX-H_Pad1.50x2.35mm_HandSolder
- J3: value SWD Connector -> SWD; footprint (none) -> Connector_PinHeader_1.00mm:PinHeader_2x05_P1.00mm_Vertical_SMD
- R1, R8: footprint Resistor_THT:R_Axial_DIN0411_L9.9mm_D3.6mm_P12.70mm_Horizontal -> Resistor_SMD:R_2512_6332Metric_Pad1.52x3.35mm_HandSolder
- SW1: value SW_Push -> Reset
- U4: value NCP1117-3.3_SOT223 -> +12V Regulator
- Y1: value Crystal_GND24 -> 8 MHz
Connections:
- net +12V: now also C1.1, J6.1
- net +3V3: no longer C1.1
- net GND: now also J6.2, J6.3
Other:
- moved on the sheet: C15

Commit message: SWD connector footprint pitch 1.0mm -> 1.27mm
Parts:
- J3: footprint Connector_PinHeader_1.00mm:PinHeader_2x05_P1.00mm_Vertical_SMD -> Connector_PinHeader_1.27mm:PinHeader_2x05_P1.27mm_Vertical_SMD
Changed lines of the file:
@@
 F 0 "J3" H 1950 2417 50  0000 C CNN
 F 1 "SWD" H 1950 2326 50  0000 C CNN
-F 2 "Connector_PinHeader_1.00mm:PinHeader_2x05_P1.00mm_Vertical_SMD" H 1900 2000 50  0001 C CNN
+F 2 "Connector_PinHeader_1.27mm:PinHeader_2x05_P1.27mm_Vertical_SMD" H 1900 2000 50  0001 C CNN
 F 3 "~" H 1900 2000 50  0001 C CNN
 	1    1900 2000
